Commit message: fixed pr2 apartment because main broke it

File: pycram/demos/bachelor_thesis/own_environments/modified_apartment.urdf (robot description, URDF)
Before this commit: robot apartment, 92 links, 91 joints
Links:
- removed link cabinet10_drawer_bottom
- removed link cabinet10_drawer_middle
- removed link cabinet10_drawer_top
- removed link cabinet11_drawer_bottom
- removed link cabinet11_drawer_middle
- removed link cabinet11_drawer_top
- removed link cabinet1_drawer_bottom
- removed link cabinet1_drawer_middle
- removed link cabinet2_drawer_big
- removed link cabinet2_drawer_small
- removed link cabinet5_drawer_bottom
- removed link cabinet5_drawer_middle
- removed link cabinet5_drawer_top
- removed link cabinet6_drawer_bottom
- removed link cabinet6_drawer_middle
- removed link cabinet6_drawer_top
- removed link cabinet8_drawer_bottom
- removed link cabinet8_drawer_middle
- removed link cabinet9_drawer_bottom
- removed link cabinet9_drawer_middle
- removed link cabinet9_drawer_top
- removed link coffee_table_drawer
- removed link dishwasher_drawer_middle
- removed link handle_cab10_b
- removed link handle_cab10_m
- removed link handle_cab10_t
- removed link handle_cab11_b
- removed link handle_cab11_m
- removed link handle_cab11_t
- removed link handle_cab1_drawer_bottom
- removed link handle_cab1_drawer_mid
- removed link handle_cab5_b
- removed link handle_cab5_m
- removed link handle_cab5_t
- removed link handle_cab6_b
- removed link handle_cab6_m
- removed link handle_cab6_t
- removed link handle_cab7_middle
- removed link handle_cab8
- removed link handle_cab9_b
- removed link handle_cab9_m
- removed link handle_cab9_t
Joints:
- removed joint cabinet10_drawer_bottom_joint
- removed joint cabinet10_drawer_middle_joint
- removed joint cabinet10_drawer_top_joint
- removed joint cabinet11_drawer_bottom_joint
- removed joint cabinet11_drawer_middle_joint
- removed joint cabinet11_drawer_top_joint
- removed joint cabinet1_drawer_bottom_joint
- removed joint cabinet1_drawer_middle_joint
- removed joint cabinet2_drawer_big_joint
- removed joint cabinet2_drawer_small_joint
- removed joint cabinet5_drawer_bottom_joint
- removed joint cabinet5_drawer_middle_joint
- removed joint cabinet5_drawer_top_joint
- removed joint cabinet6_drawer_bottom_joint
- removed joint cabinet6_drawer_middle_joint
- removed joint cabinet6_drawer_top_joint
- removed joint cabinet8_drawer_bottom_joint
- removed joint cabinet8_drawer_middle_joint
- removed joint cabinet9_drawer_bottom_joint
- removed joint cabinet9_drawer_middle_joint
- removed joint cabinet9_drawer_top_joint
- removed joint coffee_table_drawer_joint
- removed joint dishwasher_drawer_middle_joint
- removed joint handle_cab10_bott_joint
- removed joint handle_cab10_mid_joint
- removed joint handle_cab10_top_joint
- removed joint handle_cab11_bott_joint
- removed joint handle_cab11_mid_joint
- removed joint handle_cab11_top_joint
- removed joint handle_cab1_drawer_bottom_joint
- removed joint handle_cab1_drawer_mid_joint
- removed joint handle_cab5_bott_joint
- removed joint handle_cab5_mid_joint
- removed joint handle_cab5_top_joint
- removed joint handle_cab6_bott_joint
- removed joint handle_cab6_mid_joint
- removed joint handle_cab6_top_joint
- removed joint handle_cab7_drawer_middle_joint
- removed joint handle_cab8_top_joint
- removed joint handle_cab9_bott_joint
- removed joint handle_cab9_mid_joint
- removed joint handle_cab9_top_joint
